Commit message: update wx250s leader

File: open_manipulator_description/ros2_control/wx250s_leader.ros2_control.xacro (robot description, xacro)
@@ -19,5 +19,5 @@
             <param name="port_name">${port_name}</param>
             <param name="baud_rate">1000000</param>
-            <param name="error_timeout_ms">500</param>
+            <param name="error_timeout_ms">1000</param>
             <param name="dynamixel_model_folder">/param/dxl_model</param>
             <param name="number_of_joints">7</param>
@@ -105,5 +105,4 @@
         <state_interface name="Present Position"/>
         <state_interface name="Present Velocity"/>
-        <state_interface name="Present Current"/>
         <param name="Torque Enable">0</param>
       </gpio>
@@ -114,5 +113,4 @@
         <state_interface name="Present Position"/>
         <state_interface name="Present Velocity"/>
-        <state_interface name="Present Current"/>
         <param name="Torque Enable">0</param>
       </gpio>
@@ -123,5 +121,4 @@
         <state_interface name="Present Position"/>
         <state_interface name="Present Velocity"/>
-        <state_interface name="Present Current"/>
         <param name="Torque Enable">0</param>
       </gpio>
@@ -132,5 +129,4 @@
         <state_interface name="Present Position"/>
         <state_interface name="Present Velocity"/>
-        <state_interface name="Present Current"/>
         <param name="Torque Enable">0</param>
       </gpio>
@@ -141,5 +137,4 @@
         <state_interface name="Present Position"/>
         <state_interface name="Present Velocity"/>
-        <state_interface name="Present Current"/>
         <param name="Torque Enable">0</param>
       </gpio>
@@ -150,5 +145,4 @@
         <state_interface name="Present Position"/>
         <state_interface name="Present Velocity"/>
-        <state_interface name="Present Current"/>
         <param name="Torque Enable">0</param>
       </gpio>
@@ -159,5 +153,4 @@
         <state_interface name="Present Position"/>
         <state_interface name="Present Velocity"/>
-        <state_interface name="Present Current"/>
         <param name="Torque Enable">0</param>
       </gpio>

File: open_manipulator_description/urdf/wx250s/wx250s.urdf.xacro (robot description, xacro)
@@ -318,5 +318,5 @@
   </link>
   <joint name="wrist_angle" type="revolute">
-    <axis xyz="0 1 0"/>
+    <axis xyz="0 -1 0"/>
     <limit
       effort="${wrist_angle_limit_effort}"
